File: fortymate_rev2.kicad_pcb (KiCad board)
At the start: 2 copper layers, 247.7 x 76.2 mm, 96 parts, among them J1 Conn_01x05_Socket, SW1 SW_Push, SW10 SW_Push, SW11 SW_Push, SW12 SW_Push, SW13 SW_Push, SW15 SW_Push, SW16 SW_Push, SW17 SW_Push, SW18 SW_Push, SW19 SW_Push, SW2 SW_Push, SW20 SW_Push, SW21 SW_Push, SW22 SW_Push, SW23 SW_Push, SW24 SW_Push, SW25 SW_Push, SW26 SW_Push, SW29 SW_Push, SW3 SW_Push, SW30 SW_Push, SW31 SW_Push, SW32 SW_Push, SW33 SW_Push, SW34 SW_Push, SW35 SW_Push, SW36 SW_Push, SW37 SW_Push, SW38 SW_Push, SW39 SW_Push, SW4 SW_Push, SW40 SW_Push, SW43 SW_Push, SW44 SW_Push, SW45 SW_Push, SW46 SW_Push, SW47 SW_Push, SW48 SW_Push, SW5 SW_Push, SW50 SW_SPDT, SW51 SW_Push, SW6 SW_Push, SW7 SW_Push, SW8 SW_Push, SW9 SW_Push, U1 Micon_BLEMicroPro

Commit message: PCB progress + submodulized salicylic lib
Parts:
- moved BT1 4.13 mm to (218.4, 19.1), turned to -160 degrees
- moved BT2 1.75 mm to (237.5, 19.1), turned to -160 degrees
Routing:
- net (no net): track 423.1 -> 0.00 mm
- net row6: track 0.00 -> 147.6 mm
- net col4: track 10.2 -> 107.9 mm, vias 0 -> 2
- net col3: track 10.2 -> 106.1 mm, vias 1 -> 2
- net col2: track 10.2 -> 106.1 mm, vias 1 -> 2
- net col0: track 56.9 -> 104.8 mm, vias 3 -> 4
- net col6: track 5.12 -> 53.0 mm, vias 0 -> 1
- net col5: track 10.2 -> 58.2 mm, vias 0 -> 2
- net col1: track 64.0 -> 111.8 mm, vias 12 -> 4

Commit message: more pcb progress
Parts:
- removed C2: C, Capacitor_SMD:C_1206_3216Metric
- C1: moved to B.Cu
- moved SWe 20.3 mm to (29.2, -1.27)
- moved D51 9.03 mm to (237.5, 12.7), turned to 0 degrees
- moved D50 7.68 mm to (218.4, 12.7), turned to 0 degrees
- moved C1 4.14 mm to (12.7, 19.1)
- renumbered SW51 to SWe
Routing:
- net col4: track 107.9 -> 340.9 mm, vias 2 -> 9
- net col5: track 58.2 -> 284.6 mm, vias 2 -> 7
- net col3: track 106.1 -> 318.3 mm, vias 2 -> 9
- net col2: track 106.1 -> 315.6 mm, vias 2 -> 9
- net col1: track 111.8 -> 304.0 mm, vias 4 -> 10
- net col0: track 104.8 -> 276.0 mm, vias 4 -> 6
- net BAT+: track 0.00 -> 16.2 mm
- net col6: track 53.0 -> 58.7 mm, vias 1 -> 3
