File: fortymate_rev2.kicad_sch (KiCad schematic)
At the start: 96 parts, among them J1 Conn_01x05_Socket, SW1 SW_Push, SW10 SW_Push, SW11 SW_Push, SW12 SW_Push, SW13 SW_Push, SW15 SW_Push, SW16 SW_Push, SW17 SW_Push, SW18 SW_Push, SW19 SW_Push, SW2 SW_Push, SW20 SW_Push, SW21 SW_Push, SW22 SW_Push, SW23 SW_Push, SW24 SW_Push, SW25 SW_Push, SW26 SW_Push, SW29 SW_Push, SW3 SW_Push, SW30 SW_Push, SW31 SW_Push, SW32 SW_Push, SW33 SW_Push, SW34 SW_Push, SW35 SW_Push, SW36 SW_Push, SW37 SW_Push, SW38 SW_Push, SW39 SW_Push, SW4 SW_Push, SW40 SW_Push, SW43 SW_Push, SW44 SW_Push, SW45 SW_Push, SW46 SW_Push, SW47 SW_Push, SW48 SW_Push, SW5 SW_Push, SW50 SW_SPDT, SW51 SW_Push, SW6 SW_Push, SW7 SW_Push, SW8 SW_Push, SW9 SW_Push, U1 Micon_BLEMicroPro

Commit message: more pcb progress
Parts:
- removed C2: C, Capacitor_SMD:C_1206_3216Metric, symbol Device:C
Other:
- moved on the sheet: C1
Changed lines of the file:
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@@
   (junction (at 31.75 78.74) (diameter 0) (color 0 0 0 0)
   )
-  (junction (at 154.94 158.75) (diameter 0) (color 0 0 0 0)
-  )
   (junction (at 201.93 59.69) (diameter 0) (color 0 0 0 0)
   )
@@
   )
   (junction (at 168.91 41.91) (diameter 0) (color 0 0 0 0)
-  )
-  (junction (at 154.94 151.13) (diameter 0) (color 0 0 0 0)
   )
   (junction (at 74.93 104.14) (diameter 0) (color 0 0 0 0)
@@
     (stroke (width 0) (type default))
   )
-  (wire (pts (xy 148.59 151.13) (xy 154.94 151.13))
-    (stroke (width 0) (type default))
-  )
   (wire (pts (xy 212.09 85.09) (xy 228.6 85.09))
     (stroke (width 0) (type default))
@@
   )
   (wire (pts (xy 48.26 78.74) (xy 48.26 96.52))
-    (stroke (width 0) (type default))
-  )
-  (wire (pts (xy 148.59 158.75) (xy 154.94 158.75))
     (stroke (width 0) (type default))
   )
@@
     )
   )
-  (symbol (lib_id "Device:C") (at 148.59 154.94 0) (unit 1)
-    (in_bom yes) (on_board yes) (dnp no) (fields_autoplaced)
-    (property "Reference" "C1" (at 152.4 154.305 0)
+  (symbol (lib_id "Device:C") (at 154.94 154.94 0) (unit 1)
+    (in_bom yes) (on_board yes) (dnp no) (fields_autoplaced)
+    (property "Reference" "C1" (at 158.75 154.305 0)
       (effects (font (size 1.27 1.27)) (justify left))
     )
-    (property "Value" "C" (at 152.4 156.845 0)
+    (property "Value" "C" (at 158.75 156.845 0)
       (effects (font (size 1.27 1.27)) (justify left))
     )
-    (property "Footprint" "Capacitor_SMD:C_1206_3216Metric" (at 149.5552 158.75 0)
-      (effects (font (size 1.27 1.27)) hide)
-    )
-    (property "Datasheet" "~" (at 148.59 154.94 0)
+    (property "Footprint" "Capacitor_SMD:C_1206_3216Metric" (at 155.9052 158.75 0)
+      (effects (font (size 1.27 1.27)) hide)
+    )
+    (property "Datasheet" "~" (at 154.94 154.94 0)
       (effects (font (size 1.27 1.27)) hide)
     )
@@
         )
       )
-    )
-  )
-  (symbol (lib_id "Device:C") (at 154.94 154.94 0) (unit 1)
-    (in_bom yes) (on_board yes) (dnp no) (fields_autoplaced)
-    (property "Reference" "C2" (at 158.75 154.305 0)
-      (effects (font (size 1.27 1.27)) (justify left))
-    )
-    (property "Value" "C" (at 158.75 156.845 0)
-      (effects (font (size 1.27 1.27)) (justify left))
-    )
-    (property "Footprint" "Capacitor_SMD:C_1206_3216Metric" (at 155.9052 158.75 0)
-      (effects (font (size 1.27 1.27)) hide)
-    )
-    (property "Datasheet" "~" (at 154.94 154.94 0)
-      (effects (font (size 1.27 1.27)) hide)
-    )
-    (pin "1")
-    (pin "2")
-    (instances
-      (project "fortymate_rev2"
-        (path "/6f59cb56-7d85-47bf-9784-8d6ac3969dce"
-          (reference "C2") (unit 1)
-        )
-      )
